File: NTR-Subcard.kicad_pcb (KiCad board)
At the start: 2 copper layers, 22 x 18 mm, 6 parts, among them CN1 Conn_01x40_Pin, U1 M95256-WMN6P, U2 M45PE20-VMN6P

Commit message: Updates after first production batch
Signed-off-by: rosaage <tagemellemstrand@hotmail.com>
Parts:
- CN1: value Conn_01x40_Pin -> Molex_SlimStack_53748-0408_2x20_P0.50mm
- R1: value R -> 10k
- U1: value M95256-WMN6P -> M95512-WMN6P
- U2: footprint Package_SO:SOIC-8_3.9x4.9mm_P1.27mm -> tage:SOIC-8_3.9x3.9-7.62mm_P1.27mm
- moved U2 0.78 mm to (113.0, 76.2)
Routing:
- net S: track 43.7 -> 44.6 mm
Other:
- board text added: "JLCJLCJLCJLC"
